File: main/MIDI-IN.sch (KiCad schematic (older format))
At the start: 5 parts, among them J1 DIN-5_180degree, U1 6N138

Commit message: Final cleanup before sending in for rebiew
Parts:
- renumbered J1 to J2, R1 to R6, R2 to R7
Changed lines of the file:
@@
 	3950 5250 7650 5250
 $Comp
-L power:GND #PWR01
+L power:GND #PWR04
 U 1 1 61403610
 P 4400 4300
-F 0 "#PWR01" H 4400 4050 50  0001 C CNN
+F 0 "#PWR04" H 4400 4050 50  0001 C CNN
 F 1 "GND" H 4405 4127 50  0000 C CNN
 F 2 "" H 4400 4300 50  0001 C CNN
@@
 $EndComp
 $Comp
-L Device:R R1
+L Device:R R6
 U 1 1 6140361C
 P 5200 4450
-F 0 "R1" V 4993 4450 50  0000 C CNN
+F 0 "R6" V 4993 4450 50  0000 C CNN
 F 1 "220" V 5084 4450 50  0000 C CNN
 F 2 "" V 5130 4450 50  0001 C CNN
@@
 Connection ~ 5650 4450
 $Comp
-L power:GND #PWR02
+L power:GND #PWR05
 U 1 1 61403633
 P 6750 5000
-F 0 "#PWR02" H 6750 4750 50  0001 C CNN
+F 0 "#PWR05" H 6750 4750 50  0001 C CNN
 F 1 "GND" H 6755 4827 50  0000 C CNN
 F 2 "" H 6750 5000 50  0001 C CNN
@@
 	6650 4750 6900 4750
 $Comp
-L Device:R R2
+L Device:R R7
 U 1 1 6140363C
 P 6900 4600
-F 0 "R2" H 6970 4646 50  0000 L CNN
+F 0 "R7" H 6970 4646 50  0000 L CNN
 F 1 "220" H 6970 4555 50  0000 L CNN
 F 2 "" V 6830 4600 50  0001 C CNN
@@
 MIDI_IN
 $Comp
-L Connector:DIN-5_180degree J1
+L Connector:DIN-5_180degree J2
 U 1 1 6146F928
 P 4400 4000
-F 0 "J1" H 4400 3633 50  0000 C CNN
+F 0 "J2" H 4400 3633 50  0000 C CNN
 F 1 "DIN-5_180degree" H 4400 3724 50  0000 C CNN
 F 2 "" H 4400 4000 50  0001 C CNN
@@
 $EndComp
 $Comp
-L power:+3.3V #PWR0104
+L power:+3.3V #PWR06
 U 1 1 6148E544
 P 6900 4200
-F 0 "#PWR0104" H 6900 4050 50  0001 C CNN
+F 0 "#PWR06" H 6900 4050 50  0001 C CNN
 F 1 "+3.3V" H 6915 4373 50  0000 C CNN
 F 2 "" H 6900 4200 50  0001 C CNN

Commit message: Fix up after review
Done:
- Add bulk decoupling capacitor to switch regulator cirucit
- Disconnect DONE from PROGRAM_B in FPGA (mistake)
- The decoupling capacitors used for the FPGA were for the 15T, not the
  100T. It was also setup for two I/O banks, we only use one. Disconnect
  I/O bank 15.
- Switch external clock on the MCU to an oscillator, allowing for 72MHz
- Switch pinout of the backup SPI on the MCU so that half the pins are
  ground

Mizzing:
- Add low-pass filters to the output of the DAC as per the datasheet.
  May remove the need for the amplifier circuit.
Parts:
- J2: footprint (none) -> 671-0501:671-0501
- R6, R7: footprint (none) -> Resistor_SMD:R_0805_2012Metric_Pad1.20x1.40mm_HandSolder
Changed lines of the file:
@@
 	3950 5250 7650 5250
 $Comp
-L power:GND #PWR04
+L power:GND #PWR05
 U 1 1 61403610
 P 4400 4300
-F 0 "#PWR04" H 4400 4050 50  0001 C CNN
+F 0 "#PWR05" H 4400 4050 50  0001 C CNN
 F 1 "GND" H 4405 4127 50  0000 C CNN
 F 2 "" H 4400 4300 50  0001 C CNN
@@
 F 0 "R6" V 4993 4450 50  0000 C CNN
 F 1 "220" V 5084 4450 50  0000 C CNN
-F 2 "" V 5130 4450 50  0001 C CNN
+F 2 "Resistor_SMD:R_0805_2012Metric_Pad1.20x1.40mm_HandSolder" V 5130 4450 50  0001 C CNN
 F 3 "~" H 5200 4450 50  0001 C CNN
 	1    5200 4450
@@
 Connection ~ 5650 4450
 $Comp
-L power:GND #PWR05
+L power:GND #PWR06
 U 1 1 61403633
 P 6750 5000
-F 0 "#PWR05" H 6750 4750 50  0001 C CNN
+F 0 "#PWR06" H 6750 4750 50  0001 C CNN
 F 1 "GND" H 6755 4827 50  0000 C CNN
 F 2 "" H 6750 5000 50  0001 C CNN
@@
 F 0 "R7" H 6970 4646 50  0000 L CNN
 F 1 "220" H 6970 4555 50  0000 L CNN
-F 2 "" V 6830 4600 50  0001 C CNN
+F 2 "Resistor_SMD:R_0805_2012Metric_Pad1.20x1.40mm_HandSolder" V 6830 4600 50  0001 C CNN
 F 3 "~" H 6900 4600 50  0001 C CNN
 	1    6900 4600
@@
 F 0 "J2" H 4400 3633 50  0000 C CNN
 F 1 "DIN-5_180degree" H 4400 3724 50  0000 C CNN
-F 2 "" H 4400 4000 50  0001 C CNN
+F 2 "671-0501:671-0501" H 4400 4000 50  0001 C CNN
 F 3 "http://www.mouser.com/ds/2/18/40_c091_abd_e-75918.pdf" H 4400 4000 50  0001 C CNN
 	1    4400 4000
@@
 $EndComp
 $Comp
-L power:+3.3V #PWR06
+L power:+3.3V #PWR04
 U 1 1 6148E544
 P 6900 4200
-F 0 "#PWR06" H 6900 4050 50  0001 C CNN
+F 0 "#PWR04" H 6900 4050 50  0001 C CNN
 F 1 "+3.3V" H 6915 4373 50  0000 C CNN
 F 2 "" H 6900 4200 50  0001 C CNN

Commit message: DAC: Remove amplifier, replace with low pass as per datasheet
Also: a lot of footprint association
Parts:
- U1: footprint (none) -> 6N138SMT_R:SOP254P1030X460-8N
Changed lines of the file:
@@
 $Descr A4 11693 8268
 encoding utf-8
-Sheet 2 7
+Sheet 2 6
 Title "MIDI Audio Box"
 Date "2021-09-21"
@@
 F 0 "U1" H 6350 5117 50  0000 C CNN
 F 1 "6N138" H 6350 5026 50  0000 C CNN
-F 2 "" H 6640 4350 50  0001 C CNN
+F 2 "6N138SMT_R:SOP254P1030X460-8N" H 6640 4350 50  0001 C CNN
 F 3 "http://www.onsemi.com/pub/Collateral/HCPL2731-D.pdf" H 6640 4350 50  0001 C CNN
 	1    6350 4650

Commit message: Start PCB layout
Parts:
- D1: footprint Diode_THT:D_DO-35_SOD27_P7.62mm_Horizontal -> Diode_SMD:D_SOD-123F; Manufacturer_Name (none) -> Taiwan Semiconductor; Manufacturer_Part_Number (none) -> 1N4148W RH; URL (none) -> https://no.farnell.com/taiwan-semiconductor/1n4148w-rh/diod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
- J2: Manufacturer_Name (none) -> Deltron Components; Manufacturer_Part_Number (none) -> 671-0501; URL (none) -> https://no.farnell.com/deltron-components/671-0501/din-audi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
- U1: Description (none) -> Optocoupler for MIDI circuit; Manufacturer_Name (none) -> Isocom; Manufacturer_Part_Number (none) -> 6N138SMT/R; URL (none) -> https://www.digikey.no/product-detail/no/isocom-components-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
Changed lines of the file:
@@
 F 0 "D1" V 5604 4680 50  0000 L CNN
 F 1 "1N4148" V 5695 4680 50  0000 L CNN
-F 2 "Diode_THT:D_DO-35_SOD27_P7.62mm_Horizontal" H 5650 4425 50  0001 C CNN
+F 2 "Diode_SMD:D_SOD-123F" H 5650 4425 50  0001 C CNN
 F 3 "https://assets.nexperia.com/documents/data-sheet/1N4148_1N4448.pdf" H 5650 4600 50  0001 C CNN
+F 4 "Taiwan Semiconductor" H 5650 4600 50  0001 C CNN "Manufacturer_Name"
+F 5 "1N4148W RH" H 5650 4600 50  0001 C CNN "Manufacturer_Part_Number"
+F 6 "https://no.farnell.com/taiwan-semiconductor/1n4148w-rh/diode-small-sig-300v-0-15a-sod/dp/2677464?st=1n4148" H 5650 4600 50  0001 C CNN "URL"
 	1    5650 4600
 	0    1    1    0
@@
 F 1 "6N138" H 6350 5026 50  0000 C CNN
 F 2 "6N138SMT_R:SOP254P1030X460-8N" H 6640 4350 50  0001 C CNN
-F 3 "http://www.onsemi.com/pub/Collateral/HCPL2731-D.pdf" H 6640 4350 50  0001 C CNN
+F 3 "http://isocom.com/wp-content/uploads/2017/08/dc93135.pdf" H 6640 4350 50  0001 C CNN
+F 4 "Optocoupler for MIDI circuit" H 6350 4650 50  0001 C CNN "Description"
+F 5 "Isocom" H 6350 4650 50  0001 C CNN "Manufacturer_Name"
+F 6 " 6N138SMT/R " H 6350 4650 50  0001 C CNN "Manufacturer_Part_Number"
+F 7 "https://www.digikey.no/product-detail/no/isocom-components-2004-ltd/6N138SMT-R/6N138SMCT-ND/5037087" H 6350 4650 50  0001 C CNN "URL"
 	1    6350 4650
 	1    0    0    -1
@@
 F 1 "DIN-5_180degree" H 4400 3724 50  0000 C CNN
 F 2 "671-0501:671-0501" H 4400 4000 50  0001 C CNN
-F 3 "http://www.mouser.com/ds/2/18/40_c091_abd_e-75918.pdf" H 4400 4000 50  0001 C CNN
+F 3 "https://www.dem-uk.com/deltron-components/Data/Product_Downloads/deltron-671-0401-4-way-din-socket-data.pdf" H 4400 4000 50  0001 C CNN
+F 4 "Deltron Components" H 4400 4000 50  0001 C CNN "Manufacturer_Name"
+F 5 "671-0501" H 4400 4000 50  0001 C CNN "Manufacturer_Part_Number"
+F 6 "https://no.farnell.com/deltron-components/671-0501/din-audio-video-conn-jack-5pos/dp/2989966?st=din" H 4400 4000 50  0001 C CNN "URL"
 	1    4400 4000
 	-1   0    0    1
