File: main/FPGA.sch (KiCad schematic (older format))
At the start: 50 parts, among them IC3 ESP-PSRAM64H, J4 FPGA_debug, J5 FPGA_GPIO, U2 S25FL127S, U3 XC7A100T-FTG256, X1 FGPA_Oscillator

Commit message: PCB getting close to being fully connected
Still missing the power circuit, will look at it tomorrow.
Connections:
- net +3V3: now also J5.1 (Pin_1)
- net GND: now also J5.2 (Pin_2)
- net GPIO0: now also J5.3 (Pin_3), U3.R5 (IO_L23P_T3_A03_D19_14); no longer J5.1 (Pin_1), U3.R7 (IO_L24N_T3_A00_D16_14)
- net GPIO1: now also J5.5 (Pin_5), U3.T7 (IO_L21P_T3_DQS_14); no longer J5.3 (Pin_3), U3.R6 (IO_L24P_T3_A01_D17_14)
- net GPIO2: now also J5.7 (Pin_7), U3.T9 (IO_L22P_T3_A05_D21_14); no longer J5.5 (Pin_5), U3.T5 (IO_L23N_T3_A02_D18_14)
- net GPIO3: now also J5.9 (Pin_9), U3.T12 (IO_L15N_T2_DQS_DOUT_CSO_B_14); no longer J5.7 (Pin_7), U3.R5 (IO_L23P_T3_A03_D19_14)
- net GPIO4: now also J5.10 (Pin_10); no longer J5.9 (Pin_9)
- net GPIO5: now also J5.8 (Pin_8), U3.T8 (IO_L21N_T3_DQS_A06_D22_14); no longer J5.10 (Pin_10), U3.T9 (IO_L22P_T3_A05_D21_14)
- net GPIO6: now also J5.6 (Pin_6), U3.T5 (IO_L23N_T3_A02_D18_14); no longer J5.8 (Pin_8), U3.T8 (IO_L21N_T3_DQS_A06_D22_14)
- net GPIO7: now also J5.4 (Pin_4), U3.R6 (IO_L24P_T3_A01_D17_14); no longer J5.6 (Pin_6), U3.T7 (IO_L21P_T3_DQS_14)
- net GPIO8: no longer names the net of U3.R8 (IO_L20N_T3_A07_D23_14)
- net GPIO8: no longer J5.4 (Pin_4)
- net GPIO9: no longer names the net of U3.P8 (IO_L20P_T3_A08_D24_14)
- net GPIO9: no longer J5.2 (Pin_2)
- no-connect marks 142 -> 144
Changed lines of the file:
@@
 NoConn ~ 11900 5550
 NoConn ~ 11900 4850
-NoConn ~ 11900 4750
 NoConn ~ 11900 4650
 NoConn ~ 11900 4550
@@
 NoConn ~ 15900 2050
 Wire Wire Line
-	13100 7500 12800 7500
-Entry Wire Line
-	12700 7600 12800 7500
-Wire Wire Line
-	13100 7600 12800 7600
-Entry Wire Line
-	12700 7700 12800 7600
-Wire Wire Line
 	13100 7700 12800 7700
 Entry Wire Line
@@
 Entry Wire Line
 	13900 7600 14000 7700
-Entry Wire Line
-	13900 7500 14000 7600
+Text Label 13050 7700 2    50   ~ 0
+GPIO6
 Text Label 13050 7800 2    50   ~ 0
-GPIO6
+GPIO5
 Text Label 13050 7900 2    50   ~ 0
-GPIO5
+GPIO4
 Text Label 13650 7900 0    50   ~ 0
-GPIO4
+GPIO3
 Text Label 13650 7800 0    50   ~ 0
-GPIO3
+GPIO2
 Text Label 13650 7700 0    50   ~ 0
-GPIO2
+GPIO1
 Text Label 13650 7600 0    50   ~ 0
-GPIO1
-Text Label 13650 7500 0    50   ~ 0
 GPIO0
-Wire Wire Line
-	13600 7500 13900 7500
-Text Label 13050 7700 2    50   ~ 0
+Text Label 13050 7600 2    50   ~ 0
 GPIO7
-Text Label 13050 7600 2    50   ~ 0
-GPIO8
-Text Label 13050 7500 2    50   ~ 0
-GPIO9
 Text Label 12400 7350 2    50   ~ 0
 GPIO[0..9]
@@
 	9600 5500 10900 5500
 Entry Wire Line
-	11450 5850 11550 5750
-Entry Wire Line
 	11450 5950 11550 5850
 Entry Wire Line
@@
 	11450 6550 11550 6450
 Entry Wire Line
-	11450 6650 11550 6550
-Entry Wire Line
-	11450 5750 11550 5650
+	11450 6650 11350 6550
 Wire Bus Line
 	11450 7350 12700 7350
-Text Label 11600 6550 0    50   ~ 0
+Text Label 11150 6550 0    50   ~ 0
+GPIO3
+Text Label 11600 6450 0    50   ~ 0
+GPIO7
+Text Label 11600 6350 0    50   ~ 0
+GPIO6
+Text Label 11600 6250 0    50   ~ 0
 GPIO0
-Text Label 11600 6450 0    50   ~ 0
-GPIO1
-Text Label 11600 6350 0    50   ~ 0
-GPIO2
-Text Label 11600 6250 0    50   ~ 0
-GPIO3
 Text Label 11600 6150 0    50   ~ 0
 GPIO4
 Text Label 11600 6050 0    50   ~ 0
+GPIO2
+Text Label 11600 5950 0    50   ~ 0
 GPIO5
-Text Label 11600 5950 0    50   ~ 0
-GPIO6
 Text Label 11600 5850 0    50   ~ 0
-GPIO7
-Text Label 11600 5750 0    50   ~ 0
-GPIO8
-Text Label 11600 5650 0    50   ~ 0
-GPIO9
+GPIO1
 Wire Wire Line
 	7700 9850 9700 9850
@@
 	10400 3450 9800 3450
 Wire Wire Line
-	11550 6550 11900 6550
-Wire Wire Line
 	11550 6450 11900 6450
 Wire Wire Line
@@
 Wire Wire Line
 	11550 5850 11900 5850
-Wire Wire Line
-	11900 5750 11550 5750
-Wire Wire Line
-	11550 5650 11900 5650
 Wire Wire Line
 	9550 10700 9650 10700
@@
 Wire Wire Line
 	10800 4950 11900 4950
-$Comp
-L FPGA_Xilinx_Artix7:XC7A100T-FTG256 U3
-U 1 1 61604A2B
-P 13900 3850
-F 0 "U3" H 13900 6550 50  0000 C CNN
-F 1 "XC7A100T-FTG256" H 13900 900 50  0000 C CNN
-F 2 "Package_BGA:Xilinx_FTG256" H 13900 3850 50  0001 C CNN
-F 3 "https://www.google.com/url?sa=t&rct=j&q=&esrc=s&source=web&cd=&cad=rja&uact=8&ved=2ahUKEwiH1rrnlZ_zAhUrtYsKHcsIDFQQFnoECAUQAQ&url=https%3A%2F%2Fwww.xilinx.com%2Fsupport%2Fdocumentation%2Fuser_guides%2Fug475_7Series_Pkg_Pinout.pdf&usg=AOvVaw3NyLHDtSbZv1hXp1wxMn0l" H 13900 3850 50  0000 C CNN
-F 4 "Xilinx" H 13900 3850 50  0001 C CNN "Manufacturer_Name"
-F 5 "XC7A100T-FTG256" H 13900 3850 50  0001 C CNN "Manufacturer_Part_Number"
-	1    13900 3850
-	1    0    0    -1
-$EndComp
 NoConn ~ 11900 4350
 Wire Wire Line
@@
 	1    0    0    -1
 $EndComp
+Wire Wire Line
+	11900 4750 11700 4750
+Wire Wire Line
+	11700 4750 11700 5300
+Wire Wire Line
+	11700 5300 11100 5300
+Wire Wire Line
+	11100 5300 11100 6550
+Wire Wire Line
+	11100 6550 11350 6550
+$Comp
+L FPGA_Xilinx_Artix7:XC7A100T-FTG256 U3
+U 1 1 61604A2B
+P 13900 3850
+F 0 "U3" H 13900 6550 50  0000 C CNN
+F 1 "XC7A100T-FTG256" H 13900 900 50  0000 C CNN
+F 2 "Package_BGA:Xilinx_FTG256" H 13900 3850 50  0001 C CNN
+F 3 "https://www.google.com/url?sa=t&rct=j&q=&esrc=s&source=web&cd=&cad=rja&uact=8&ved=2ahUKEwiH1rrnlZ_zAhUrtYsKHcsIDFQQFnoECAUQAQ&url=https%3A%2F%2Fwww.xilinx.com%2Fsupport%2Fdocumentation%2Fuser_guides%2Fug475_7Series_Pkg_Pinout.pdf&usg=AOvVaw3NyLHDtSbZv1hXp1wxMn0l" H 13900 3850 50  0000 C CNN
+F 4 "Xilinx" H 13900 3850 50  0001 C CNN "Manufacturer_Name"
+F 5 "XC7A100T-FTG256" H 13900 3850 50  0001 C CNN "Manufacturer_Part_Number"
+	1    13900 3850
+	1    0    0    -1
+$EndComp
+NoConn ~ 11900 6550
+NoConn ~ 11900 5650
+NoConn ~ 11900 5750
+Entry Wire Line
+	12800 7600 12700 7700
+Wire Wire Line
+	12800 7600 13100 7600
+$Comp
+L power:+3.3V #PWR0101
+U 1 1 617E6C6F
+P 13700 7350
+F 0 "#PWR0101" H 13700 7200 50  0001 C CNN
+F 1 "+3.3V" H 13715 7523 50  0000 C CNN
+F 2 "" H 13700 7350 50  0001 C CNN
+F 3 "" H 13700 7350 50  0001 C CNN
+	1    13700 7350
+	-1   0    0    -1
+$EndComp
+Wire Wire Line
+	13700 7350 13700 7500
+Wire Wire Line
+	13700 7500 13600 7500
+$Comp
+L power:GND #PWR0102
+U 1 1 61811D03
+P 13000 7350
+F 0 "#PWR0102" H 13000 7100 50  0001 C CNN
+F 1 "GND" H 13005 7177 50  0000 C CNN
+F 2 "" H 13000 7350 50  0001 C CNN
+F 3 "" H 13000 7350 50  0001 C CNN
+	1    13000 7350
+	1    0    0    1
+$EndComp
+Wire Wire Line
+	13000 7350 13000 7500
+Wire Wire Line
+	13000 7500 13100 7500
 Wire Bus Line
 	10250 3150 10250 3350
@@
 	12700 7350 12700 8400
 Wire Bus Line
-	14000 7600 14000 8400
+	14000 7700 14000 8400
 Wire Bus Line
-	11450 5750 11450 7350
+	11450 5950 11450 7350
 $EndSCHEMATC

Commit message: Add missing junction
Connections:
- net +3V3: now also C19.1, R18.1, R19.1, R20.1
Other:
- note added: "Junction missing in v1.0.0. \nFixed on board by soldering wire between U2 pin 8 and 3v3 pad on R19"
Changed lines of the file:
@@
 	5350 2950 5450 2950
 Wire Wire Line
-	5450 2950 5450 1600
+	5450 2950 5450 1700
 $Comp
 L power:+3.3V #PWR020
@@
 Connection ~ 4700 1700
 Wire Wire Line
-	4700 1700 5650 1700
+	4700 1700 5450 1700
 Wire Wire Line
 	8250 3100 8250 2150
@@
 Wire Wire Line
 	13000 7500 13100 7500
+Connection ~ 5450 1700
+Wire Wire Line
+	5450 1700 5450 1600
+Wire Wire Line
+	5450 1700 5650 1700
+Wire Notes Line
+	5350 1600 5550 1600
+Wire Notes Line
+	5550 1600 5550 1800
+Wire Notes Line
+	5550 1800 5350 1800
+Wire Notes Line
+	5350 1800 5350 1600
 Wire Bus Line
 	10250 3150 10250 3350
@@
 Wire Bus Line
 	11450 5950 11450 7350
+Text Notes 5600 1650 0    50   ~ 0
+Junction missing in v1.0.0. \nFixed on board by soldering wire between U2 pin 8 and 3v3 pad on R19
 $EndSCHEMATC
